Commit message: lab5

File: beginner_tutorials/urdf/myfirst.urdf (robot description, URDF)
Before this commit: robot multipleshapes, 4 links, 3 joints
Joints:
- joint link1_to_link2: origin xyz=0.026 0 0.00982 -> xyz=0 0 0.085; type fixed -> revolute
- joint link2_to_link3: origin xyz=0.138 0 0.00982 -> xyz=0.145 0 0.205; type fixed -> revolute
